Commit message: update fingereye collision to convexhull

File: FingerEyeLab/assets/xarm7_leap_right/xarm7_leap_right.urdf (robot description, URDF)
Before this commit: robot xarm7, 60 links, 59 joints
Links:
- link fingertip: geometry collision mesh filename=leap_hand_meshes/collision/soft_ring_acrylic_convex_hull.obj; visual mesh filename=leap_hand_meshes/visual/soft_ring_adjust.STL
- link fingertip_2: geometry collision mesh filename=leap_hand_meshes/collision/soft_ring_acrylic_convex_hull.obj; visual mesh filename=leap_hand_meshes/visual/soft_ring_adjust.STL
- link fingertip_3: geometry collision mesh filename=leap_hand_meshes/collision/soft_ring_acrylic_convex_hull.obj; visual mesh filename=leap_hand_meshes/visual/soft_ring_adjust.STL
- link thumb_soft_ring: geometry collision mesh filename=leap_hand_meshes/collision/soft_ring_acrylic_convex_hull.obj; visual mesh filename=leap_hand_meshes/visual/soft_ring_adjust.STL
